Commit message: gazebo+Rviz movement display

File: description/robot.urdf.xacro (robot description, xacro)
@@ -3,3 +3,4 @@
     <!-- Example link -->
     <xacro:include filename="robot_core.xacro"/>
+    <xacro:include filename="gazebo_control.xacro"/>
 </robot>

File: description/robot_core.xacro (robot description, xacro)
@@ -42,4 +42,7 @@
         </collision>
     </link>
+    <gazebo reference="chassis">
+        <material>Gazebo/White</material>
+    </gazebo>
     <!--LEFT WHEEL LINK-->
     <joint name="left_wheel_joint" type="continuous">
@@ -67,4 +70,7 @@
         </xacro:inertial_cylinder>
     </link>
+    <gazebo reference="left_wheel">
+        <material>Gazebo/Blue</material>
+    </gazebo>
     <!--RIGHT WHEEL LINK-->
     <joint name="right_wheel_joint" type="continuous">
@@ -92,4 +98,7 @@
         </xacro:inertial_cylinder>
     </link>
+    <gazebo reference="right_wheel">
+        <material>Gazebo/Blue</material>
+    </gazebo>
     <!--CASTER WHEEL FRONT RIGHT-->
     <joint name="caster_wheel_front_right_joint" type="fixed">
@@ -116,4 +125,9 @@
         </xacro:inertial_sphere>
     </link>
+    <gazebo reference="caster_wheel_front_right">
+        <material>Gazebo/Black</material>
+        <mu1 value="0.001"/>
+        <mu2 value="0.001"/>
+    </gazebo>
     <!--CASTER WHEEL FRONT LEFT-->
     <joint name="caster_wheel_front_left_joint" type="fixed">
@@ -140,4 +154,9 @@
         </xacro:inertial_sphere>
     </link>
+    <gazebo reference="caster_wheel_front_left">
+        <material>Gazebo/Black</material>
+        <mu1 value="0.001"/>
+        <mu2 value="0.001"/>
+    </gazebo>
     <!--CASTER WHEEL BACK RIGHT-->
     <joint name="caster_wheel_back_right_joint" type="fixed">
@@ -164,4 +183,9 @@
         </xacro:inertial_sphere>
     </link>
+    <gazebo reference="caster_wheel_back_right">
+        <material>Gazebo/Black</material>
+        <mu1 value="0.001"/>
+        <mu2 value="0.001"/>
+    </gazebo>
     <!--CASTER WHEEL BACK LEFT-->
     <joint name="caster_wheel_back_left_joint" type="fixed">
@@ -188,3 +212,8 @@
         </xacro:inertial_sphere>
     </link>
+    <gazebo reference="caster_wheel_back_left">
+        <material>Gazebo/Black</material>
+        <mu1 value="0.001"/>
+        <mu2 value="0.001"/>
+    </gazebo>
 </robot>

Commit message: lidar 2D scan

File: description/robot.urdf.xacro (robot description, xacro)
@@ -4,3 +4,4 @@
     <xacro:include filename="robot_core.xacro"/>
     <xacro:include filename="gazebo_control.xacro"/>
+    <xacro:include filename="lidar.xacro"/>
 </robot>

File: description/robot_core.xacro (robot description, xacro)
@@ -13,4 +13,7 @@
     <material name="black">
         <color rgba="0 0 0 1" />
+    </material>
+    <material name="red">
+        <color rgba="1 0 0 1" />
     </material>
     <!--BASE LINK-->
