Commit message: slam_toolbox integrated

File: description/lidar.xacro (robot description, xacro)
@@ -28,5 +28,5 @@
         <sensor name="laser" type="ray">
             <pose>0 0 0 0 0 0</pose>
-            <visualize>false</visualize>
+            <visualize>true</visualize>
             <update_rate>10</update_rate>
             <ray>

File: description/robot.urdf.xacro (robot description, xacro)
@@ -1,4 +1,11 @@
 <?xml version="1.0"?>
 <robot xmlns:xacro="http://www.ros.org/wiki/xacro"  name="robot">
+    <xacro:arg name="use_ros2_control" default="true"/>
+    <!-- <xacro:if value="$(arg use_ros2_control)">
+        <xacro:include filename="ros2_control.xacro" />
+    </xacro:if>
+    <xacro:unless value="$(arg use_ros2_control)">
+        <xacro:include filename="gazebo_control.xacro" />
+    </xacro:unless> -->
     <!-- Example link -->
     <xacro:include filename="robot_core.xacro"/>

File: description/robot_core.xacro (robot description, xacro)
@@ -21,4 +21,12 @@
         <!-- You can add visuals and collision properties for the base_link here if needed -->
     </link>
+    <!-- BASE_FOOTPRINT -->
+    <joint name="base_footprint_joint" type="fixed">
+        <parent link="base_link"/>
+        <child link="base_footprint"/>
+        <origin xyz="0 0 0" rpy="0 0 0"/>
+    </joint>
+    <link name="base_footprint">
+    </link>
     <!--CHASSIS LINK-->
     <joint name="chassis_joint" type="fixed">
@@ -48,166 +56,4 @@
         <material>Gazebo/White</material>
     </gazebo>
-    <!--LEFT SUPPORT-->
-    <joint name="left_support_joint" type="fixed">
-        <parent link="chassis" />
-        <child link="left_support" />
-        <origin xyz="0.2 0.25 0.15" rpy="0 0 0"/>
-    </joint>
-    <link name="left_support">
-        <xacro:inertial_box mass="0.5" x="0.05" y="0.05" z="1.5">
-            <origin xyz="0.0 0.0 0.75" rpy="0 0 0"/>
-        </xacro:inertial_box>
-        <visual>
-            <origin xyz="0.0 0.0 0.75"/>
-            <geometry>
-                <box size="0.05 0.05 1.5" />
-            </geometry>
-            <material name="orange"/>
-        </visual>
-        <collision>
-            <origin xyz="0.0 0.0 0.75"/>
-            <geometry>
-                <box size="0.05 0.05 1.5" />
-            </geometry>
-        </collision>
-    </link>
-    <gazebo reference="left_support">
-        <material>Gazebo/Orange</material>
-    </gazebo>
-    <!--RIGHT SUPPORT-->
-    <joint name="right_support_joint" type="fixed">
-        <parent link="chassis" />
-        <child link="right_support" />
-        <origin xyz="0.2 -0.25 0.15" rpy="0 0 0"/>
-    </joint>
-    <link name="right_support">
-        <xacro:inertial_box mass="0.5" x="0.05" y="0.05" z="1.5">
-            <origin xyz="0.0 0.0 0.75" rpy="0 0 0"/>
-        </xacro:inertial_box>
-        <visual>
-            <origin xyz="0.0 0.0 0.75"/>
-            <geometry>
-                <box size="0.05 0.05 1.5" />
-            </geometry>
-            <material name="orange"/>
-        </visual>
-        <collision>
-            <origin xyz="0.0 0.0 0.75"/>
-            <geometry>
-                <box size="0.05 0.05 1.5" />
-            </geometry>
-        </collision>
-    </link>
-    <gazebo reference="right_support">
-        <material>Gazebo/Orange</material>
-    </gazebo>
-    <!--SHELF 1-->
-    <joint name="shelf_1_joint" type="fixed">
-        <parent link="chassis" />
-        <child link="shelf_1" />
-        <origin xyz="0.2 0.0 1.65" rpy="0 0 0"/>
-    </joint>
-    <link name="shelf_1">
-        <xacro:inertial_box mass="0.2" x="0.3" y="0.5" z="0.05">
-            <origin xyz="0.0 0.0 0.0" rpy="0 0 0"/>
-        </xacro:inertial_box>
-        <visual>
-            <origin xyz="0.0 0.0 0.00"/>
-            <geometry>
-                <box size="0.3 0.5 0.05" />
-            </geometry>
-            <material name="orange"/>
-        </visual>
-        <collision>
-            <origin xyz="0.0 0.0 0.0"/>
-            <geometry>
-                <box size="0.3 0.5 0.05" />
-            </geometry>
-        </collision>
-    </link>
-    <gazebo reference="shelf_1">
-        <material>Gazebo/Blue</material>
-    </gazebo>
-    <!--SHELF 2-->
-    <joint name="shelf_2_joint" type="fixed">
-        <parent link="chassis" />
-        <child link="shelf_2" />
-        <origin xyz="0.2 0.0 1.3" rpy="0 0 0"/>
-    </joint>
-    <link name="shelf_2">
-        <xacro:inertial_box mass="0.2" x="0.3" y="0.5" z="0.05">
-            <origin xyz="0.0 0.0 0.0" rpy="0 0 0"/>
-        </xacro:inertial_box>
-        <visual>
-            <origin xyz="0.0 0.0 0.00"/>
-            <geometry>
-                <box size="0.3 0.5 0.05" />
-            </geometry>
-            <material name="orange"/>
-        </visual>
-        <collision>
-            <origin xyz="0.0 0.0 0.0"/>
-            <geometry>
-                <box size="0.3 0.5 0.05" />
-            </geometry>
-        </collision>
-    </link>
-    <gazebo reference="shelf_2">
-        <material>Gazebo/Blue</material>
-    </gazebo>
-    <!--SHELF 3-->
-    <joint name="shelf_3_joint" type="fixed">
-        <parent link="chassis" />
-        <child link="shelf_3" />
-        <origin xyz="0.2 0.0 0.95" rpy="0 0 0"/>
-    </joint>
-    <link name="shelf_3">
-        <xacro:inertial_box mass="0.2" x="0.3" y="0.5" z="0.05">
-            <origin xyz="0.0 0.0 0.0" rpy="0 0 0"/>
-        </xacro:inertial_box>
-        <visual>
-            <origin xyz="0.0 0.0 0.00"/>
-            <geometry>
-                <box size="0.3 0.5 0.05" />
-            </geometry>
-            <material name="orange"/>
-        </visual>
-        <collision>
-            <origin xyz="0.0 0.0 0.0"/>
-            <geometry>
-                <box size="0.3 0.5 0.05" />
-            </geometry>
-        </collision>
-    </link>
-    <gazebo reference="shelf_3">
-        <material>Gazebo/Blue</material>
-    </gazebo>
-    <!--SHELF 4-->
-    <joint name="shelf_4_joint" type="fixed">
-        <parent link="chassis" />
-        <child link="shelf_4" />
-        <origin xyz="0.2 0.0 0.6" rpy="0 0 0"/>
-    </joint>
-    <link name="shelf_4">
-        <xacro:inertial_box mass="0.2" x="0.3" y="0.5" z="0.05">
-            <origin xyz="0.0 0.0 0.0" rpy="0 0 0"/>
-        </xacro:inertial_box>
-        <visual>
-            <origin xyz="0.0 0.0 0.00"/>
-            <geometry>
-                <box size="0.3 0.5 0.05" />
-            </geometry>
-            <material name="orange"/>
-        </visual>
-        <collision>
-            <origin xyz="0.0 0.0 0.0"/>
-            <geometry>
-                <box size="0.3 0.5 0.05" />
-            </geometry>
-        </collision>
-    </link>
-    <gazebo reference="shelf_4">
-        <material>Gazebo/Blue</material>
-    </gazebo>
     <!--LEFT WHEEL LINK-->
     <joint name="left_wheel_joint" type="continuous">
@@ -228,5 +74,5 @@
             <origin xyz="0 0 0"/>
             <geometry>
-                <cylinder radius="0.07" length="0.04"/>
+                <sphere radius="0.07"/>
             </geometry>
         </collision>
@@ -256,5 +102,5 @@
             <origin xyz="0 0 0"/>
             <geometry>
-                <cylinder radius="0.07" length="0.04"/>
+                <sphere radius="0.07"/>
             </geometry>
         </collision>
@@ -292,6 +138,6 @@
     <gazebo reference="caster_wheel_front_right">
         <material>Gazebo/Black</material>
-        <mu1 value="0.001"/>
-        <mu2 value="0.001"/>
+        <mu1 value="0.0001"/>
+        <mu2 value="0.0001"/>
     </gazebo>
     <!--CASTER WHEEL FRONT LEFT-->
@@ -321,6 +167,6 @@
     <gazebo reference="caster_wheel_front_left">
         <material>Gazebo/Black</material>
-        <mu1 value="0.001"/>
-        <mu2 value="0.001"/>
+        <mu1 value="0.0001"/>
+        <mu2 value="0.0001"/>
     </gazebo>
     <!--CASTER WHEEL BACK RIGHT-->
@@ -350,6 +196,6 @@
     <gazebo reference="caster_wheel_back_right">
         <material>Gazebo/Black</material>
-        <mu1 value="0.001"/>
-        <mu2 value="0.001"/>
+        <mu1 value="0.0001"/>
+        <mu2 value="0.0001"/>
     </gazebo>
     <!--CASTER WHEEL BACK LEFT-->
@@ -379,6 +225,6 @@
     <gazebo reference="caster_wheel_back_left">
         <material>Gazebo/Black</material>
-        <mu1 value="0.001"/>
-        <mu2 value="0.001"/>
+        <mu1 value="0.0001"/>
+        <mu2 value="0.0001"/>
     </gazebo>
 </robot>
