Commit message: added functional camera

File: install/BB01/share/BB01/description/lidar.xacro (robot description, xacro)
@@ -4,5 +4,5 @@
         <parent link="chassis" />
         <child link="laser_frame" />
-        <origin xyz="0.5 0 0.175" rpy="0 0 0"/>
+        <origin xyz="0.2 0 0.175" rpy="0 0 0"/>
     </joint>
     <link name="laser_frame">
@@ -10,5 +10,5 @@
             <origin xyz="0 0 0"/>
             <geometry>
-                <cylinder radius="0.07" length="0.04"/>
+                <cylinder radius="0.02" length="0.04"/>
             </geometry>
             <material name="red"/>
@@ -28,5 +28,5 @@
         <sensor name="laser" type="ray">
             <pose>0 0 0 0 0 0</pose>
-            <visualize>false</visualize>
+            <visualize>true</visualize>
             <update_rate>10</update_rate>
             <ray>
@@ -35,6 +35,6 @@
                         <samples>270</samples>
                         <resolution>1</resolution>
-                        <min_angle>-2.3</min_angle>
-                        <max_angle>2.3</max_angle>
+                        <min_angle>-2.14</min_angle>
+                        <max_angle>2.14</max_angle>
                     </horizontal>
                 </scan>

File: install/BB01/share/BB01/description/robot.urdf.xacro (robot description, xacro)
@@ -5,4 +5,3 @@
     <xacro:include filename="gazebo_control.xacro"/>
     <xacro:include filename="lidar.xacro"/>
-    <xacro:include filename="camera.xacro"/>
 </robot>

File: install/BB01/share/BB01/description/robot_core.xacro (robot description, xacro)
@@ -26,5 +26,5 @@
         <child link="chassis"/>
         <origin xyz="-0.3 0 0"/>
-        <xacro:inertial_box mass="2.0" x="0.6" y="0.5" z="0.15">
+        <xacro:inertial_box mass="0.5" x="0.6" y="0.5" z="0.15">
             <origin xyz="0.3 0 0.075" rpy="0 0 0"/>
         </xacro:inertial_box>
@@ -49,163 +49,28 @@
     </gazebo>
     <!--LEFT SUPPORT-->
-    <joint name="left_support_joint" type="fixed">
+    <joint name="left_support_joint" type="fixed">/
         <parent link="chassis" />
         <child link="left_support" />
-        <origin xyz="0.2 0.25 0.15" rpy="0 0 0"/>
-    </joint>
-    <link name="left_support">
-        <xacro:inertial_box mass="0.5" x="0.05" y="0.05" z="1.5">
-            <origin xyz="0.0 0.0 0.75" rpy="0 0 0"/>
+        <origin xyz="0.2 -0.3 1.5" rpy="0 0 0"/>
+        <xacro:inertial_box mass="0.5" x="0.6" y="0.5" z="0.15">
+            <origin xyz="0.2 -0.3 1.5" rpy="0 0 0"/>
         </xacro:inertial_box>
-        <visual>
-            <origin xyz="0.0 0.0 0.75"/>
-            <geometry>
-                <box size="0.05 0.05 1.5" />
+    </joint>
+    <link name="left_support_joint">
+        <visual>
+            <origin xyz="0.2 -0.3 1.5"/>
+            <geometry>
+                <box size="0.2 0.2 1.5" />
             </geometry>
             <material name="orange"/>
         </visual>
         <collision>
-            <origin xyz="0.0 0.0 0.75"/>
-            <geometry>
-                <box size="0.05 0.05 1.5" />
-            </geometry>
-        </collision>
-    </link>
-    <gazebo reference="left_support">
-        <material>Gazebo/Orange</material>
-    </gazebo>
-    <!--RIGHT SUPPORT-->
-    <joint name="right_support_joint" type="fixed">
-        <parent link="chassis" />
-        <child link="right_support" />
-        <origin xyz="0.2 -0.25 0.15" rpy="0 0 0"/>
-    </joint>
-    <link name="right_support">
-        <xacro:inertial_box mass="0.5" x="0.05" y="0.05" z="1.5">
-            <origin xyz="0.0 0.0 0.75" rpy="0 0 0"/>
-        </xacro:inertial_box>
-        <visual>
-            <origin xyz="0.0 0.0 0.75"/>
-            <geometry>
-                <box size="0.05 0.05 1.5" />
-            </geometry>
-            <material name="orange"/>
-        </visual>
-        <collision>
-            <origin xyz="0.0 0.0 0.75"/>
-            <geometry>
-                <box size="0.05 0.05 1.5" />
-            </geometry>
-        </collision>
-    </link>
-    <gazebo reference="right_support">
-        <material>Gazebo/Orange</material>
-    </gazebo>
-    <!--SHELF 1-->
-    <joint name="shelf_1_joint" type="fixed">
-        <parent link="chassis" />
-        <child link="shelf_1" />
-        <origin xyz="0.2 0.0 1.65" rpy="0 0 0"/>
-    </joint>
-    <link name="shelf_1">
-        <xacro:inertial_box mass="0.2" x="0.3" y="0.5" z="0.05">
-            <origin xyz="0.0 0.0 0.0" rpy="0 0 0"/>
-        </xacro:inertial_box>
-        <visual>
-            <origin xyz="0.0 0.0 0.00"/>
-            <geometry>
-                <box size="0.3 0.5 0.05" />
-            </geometry>
-            <material name="orange"/>
-        </visual>
-        <collision>
-            <origin xyz="0.0 0.0 0.0"/>
-            <geometry>
-                <box size="0.3 0.5 0.05" />
-            </geometry>
-        </collision>
-    </link>
-    <gazebo reference="shelf_1">
-        <material>Gazebo/Blue</material>
-    </gazebo>
-    <!--SHELF 2-->
-    <joint name="shelf_2_joint" type="fixed">
-        <parent link="chassis" />
-        <child link="shelf_2" />
-        <origin xyz="0.2 0.0 1.3" rpy="0 0 0"/>
-    </joint>
-    <link name="shelf_2">
-        <xacro:inertial_box mass="0.2" x="0.3" y="0.5" z="0.05">
-            <origin xyz="0.0 0.0 0.0" rpy="0 0 0"/>
-        </xacro:inertial_box>
-        <visual>
-            <origin xyz="0.0 0.0 0.00"/>
-            <geometry>
-                <box size="0.3 0.5 0.05" />
-            </geometry>
-            <material name="orange"/>
-        </visual>
-        <collision>
-            <origin xyz="0.0 0.0 0.0"/>
-            <geometry>
-                <box size="0.3 0.5 0.05" />
-            </geometry>
-        </collision>
-    </link>
-    <gazebo reference="shelf_2">
-        <material>Gazebo/Blue</material>
-    </gazebo>
-    <!--SHELF 3-->
-    <joint name="shelf_3_joint" type="fixed">
-        <parent link="chassis" />
-        <child link="shelf_3" />
-        <origin xyz="0.2 0.0 0.95" rpy="0 0 0"/>
-    </joint>
-    <link name="shelf_3">
-        <xacro:inertial_box mass="0.2" x="0.3" y="0.5" z="0.05">
-            <origin xyz="0.0 0.0 0.0" rpy="0 0 0"/>
-        </xacro:inertial_box>
-        <visual>
-            <origin xyz="0.0 0.0 0.00"/>
-            <geometry>
-                <box size="0.3 0.5 0.05" />
-            </geometry>
-            <material name="orange"/>
-        </visual>
-        <collision>
-            <origin xyz="0.0 0.0 0.0"/>
-            <geometry>
-                <box size="0.3 0.5 0.05" />
-            </geometry>
-        </collision>
-    </link>
-    <gazebo reference="shelf_3">
-        <material>Gazebo/Blue</material>
-    </gazebo>
-    <!--SHELF 4-->
-    <joint name="shelf_4_joint" type="fixed">
-        <parent link="chassis" />
-        <child link="shelf_4" />
-        <origin xyz="0.2 0.0 0.6" rpy="0 0 0"/>
-    </joint>
-    <link name="shelf_4">
-        <xacro:inertial_box mass="0.2" x="0.3" y="0.5" z="0.05">
-            <origin xyz="0.0 0.0 0.0" rpy="0 0 0"/>
-        </xacro:inertial_box>
-        <visual>
-            <origin xyz="0.0 0.0 0.00"/>
-            <geometry>
-                <box size="0.3 0.5 0.05" />
-            </geometry>
-            <material name="orange"/>
-        </visual>
-        <collision>
-            <origin xyz="0.0 0.0 0.0"/>
-            <geometry>
-                <box size="0.3 0.5 0.05" />
-            </geometry>
-        </collision>
-    </link>
-    <gazebo reference="shelf_4">
+            <origin xyz="0.2 -0.3 1.5" />
+            <geometry>
+                <box size="0.2 0.2 1.5" />
+            </geometry>
+        </collision>
+    </link>
+    <gazebo reference="chassis">
         <material>Gazebo/Blue</material>
     </gazebo>
@@ -214,5 +79,5 @@
         <parent link="base_link"/>
         <child link="left_wheel"/>
-        <origin xyz="-0.10 0.275 0" rpy="-${pi/2} 0 0"/>
+        <origin xyz="0 0.275 0" rpy="-${pi/2} 0 0"/>
         <axis xyz="0 0 1"/>
     </joint>
@@ -242,5 +107,5 @@
         <parent link="base_link"/>
         <child link="right_wheel"/>
-        <origin xyz="-0.10 -0.275 0" rpy="${pi/2} 0 0"/>
+        <origin xyz="0 -0.275 0" rpy="${pi/2} 0 0"/>
         <axis xyz="0 0 -1"/>
     </joint>
